File: PCB/satnogs_controller/satnogs_controller.sch (KiCad schematic (older format))
At the start: 32 parts, among them P1 RS485, P2 End-Stops, P4 I2C, P5 DC Motors Driver, P6 Power-IN, P7 Motor1, P8 Motor2, P9 Dev-Pins, U1 Pro_Mini, U2 MAX485, U3 POLOLU_A4988, U4 POLOLU_A4988

Commit message: Rotator controller (#27)
* Update satnogs library.

Add new footprints, 3d shapes and schematic components.

* Updates in rotator controller.

Add RJ45 for communication and power in (PoE).
New dimensions of board (euroboard 100x80 mm)
Embed the power supply to the board (WIP).
Add pins for indicator LED and for rf switch (optional).
Add additional pads for power in case that PoE (RJ45) isn't suitable.
Updates in schematic and board wuth new library parts.

* Add PCA9540B schematic component, I2C multiplexer.

* Add fuse holder and stitching via.

* Updates in PCB and schematic.

Add digital and power ground planes (WIP).
Connection of separate GND with zero resistor.
Add I2C multiplexer.
Finalize power supply of 12V.
Change RJ45 to headers.
Add RC filter (LPF) for end-stops.
Add more dev-pins.
Add filter in uC voltage input.

Signed-off-by: zisi <agzisim@gmail.com>

* Add GND-GNDD vias and silkscreen.

Signed-off-by: zisi <agzisim@gmail.com>

* Updates according to Kicad library convention

Signed-off-by: zisi <agzisim@gmail.com>

* Resolve issues #22, #23, #24, #25

Signed-off-by: zisi <agzisim@gmail.com>

* Fix silkscreen placement and zone cleanup

* Use one GND bottom plane and GND areas in front

Remove zero ohm resistors
To avoid connection with GNDD directly with motor GND use keep out area

Signed-off-by: zisi <agzisim@gmail.com>

* Add electrolytic capacitor, TVS-diode in PSU input

Capacitor reduces the voltage ripple of input voltage (long cable)
TVS-diode protect the PSU and all the board from surges and ESD events

Signed-off-by: zisi <agzisim@gmail.com>
Parts:
- removed C2: 10u, Capacitors_ThroughHole:C_Radial_D6.3_L11.2_P2.5, symbol CP
- removed D1: ZENERsmall, Diodes_ThroughHole:Diode_DO-41_SOD81_Horizontal_RM10, symbol ZENERsmall
- removed P1: RS485, Pin_Headers:Pin_Header_Angled_1x04, symbol CONN_01X04
- removed P5: DC Motors Driver, satnogs:pin_socket_18, symbol CONN_01X18
- removed P6: Power-IN, Connect:bornier2, symbol CONN_01X02
- removed P9: Dev-Pins, Pin_Headers:Pin_Header_Straight_2x02, symbol CONN_02X02
- removed U1: Pro_Mini, satnogs:pro-mini, symbol Pro_Mini
- removed U2: MAX485, Housings_SOIC:SOIC-8_3.9x4.9mm_Pitch1.27mm, symbol MAX485
- removed U3, U4: POLOLU_A4988, satnogs:SWDIP8_.6W, symbol POLOLU_A4988
- added C10, C11, C12, C13, C14: 0.1u, Capacitors_SMD:C_0805_HandSoldering, symbol C_Small
- added C15: 100u, satnogs:CP_Radial_D10.0mm_P5.00mm, symbol CP
- added C2: 2.2u, Capacitors_SMD:C_1210_HandSoldering, symbol C_Small
- added C5: 100u, Capacitors_SMD:c_elec_6.3x5.3, symbol CP
- added C6: 100n, Capacitors_SMD:C_0805_HandSoldering, symbol C_Small
- added C7: 7.5n, Capacitors_SMD:C_0805_HandSoldering, symbol C_Small
- added C8: 10p, Capacitors_SMD:C_0805_HandSoldering, symbol C_Small
- added C9: 47u, Capacitors_SMD:C_1210_HandSoldering, symbol C_Small
- added D1, D2: D_Schottky, satnogs:DO-214AB_Handsoldering, symbol D_Schottky
- added D3: D_TVS_x2_AAC, TO_SOT_Packages_SMD:SOT-23_Handsoldering, symbol D_TVS_x2_AAC
- added D4: D_TVS, satnogs:DO-214AB_Handsoldering, symbol D_TVS
- added F1: FUSE, satnogs:FuseHolder_Keystone-3557-10, symbol FUSE
- added FB1, FB2: FILTER, Resistors_SMD:R_0805_HandSoldering, symbol FILTER
- added JP7, JP8: Jumper_NO_Small, Resistors_SMD:R_0805_HandSoldering, symbol Jumper_NO_Small
- added L1: 27u, satnogs:Inductor_Bourns-SRR1210_HandSoldering, symbol INDUCTOR_SMALL
- added P1: DEV-PINS, Pin_Headers:Pin_Header_Straight_2x04, symbol CONN_02X04
- added P3: IN-PINS, Pin_Headers:Pin_Header_Straight_2x04, symbol CONN_02X04
- added P5: GND-PAD, Mounting_Holes:MountingHole_2.2mm_M2_DIN965_Pad, symbol CONN_01X01
- added R10: 221k, Resistors_SMD:R_0805_HandSoldering, symbol R
- added R11: 26.7k, Resistors_SMD:R_0805_HandSoldering, symbol R
- added R12: 147k, Resistors_SMD:R_0805_HandSoldering, symbol R
- added R13: 10.5k, Resistors_SMD:R_0805_HandSoldering, symbol R
- added R14, R15: 200, Resistors_SMD:R_0805_HandSoldering, symbol R
- added R16, R17: 4.7k, Resistors_SMD:R_0805_HandSoldering, symbol R
- added R18: 10k, Resistors_SMD:R_0805_HandSoldering, symbol R
- added U1: Arduino_Pro_Mini, satnogs:Arduino_Pro_Mini, symbol Arduino_Pro_Mini
- added U2: SN65HVD485EDR, satnogs:SOIC-8_3.9x4.9mm_Pitch1.27mm_HandSoldering, symbol SN65HVD485EDR
- added U3, U4: Pololu_A4988, satnogs:Pololu_A4988, symbol Pololu_A4988
- added U5: TPS54360DDA, satnogs:HSOP-8, symbol TPS54360DDA
- added U6: Pololu_Dual_MC33926, satnogs:Pololu_Dual_MC33926, symbol Pololu_Dual_MC33926
- added U7: PCA9540B, satnogs:TSSOP-8_3x3mm_Pitch0.65mm_HandSoldering, symbol PCA9540B
- added U8: TC74, satnogs:SOT-23-5_HandSoldering, symbol TC74
- C1: Distributor Mouser 77-VJ0805Y104KXJCBC -> (none); Manufacturer VJ0805Y104KXJCW1BC -> (none); Mnf. (none) -> 08053C104KAT2A; Notes 16VDC -> (none); Package 0805 -> (none); Price 0.118€ -> 0.094
- C3, C4: footprint Capacitors_ThroughHole:C_Radial_D6.3_L11.2_P2.5 -> Capacitors_SMD:c_elec_6.3x5.3; Distributor Mouser 667-ECA-1VM101 -> (none); Manufacturer ECA-1VM101 -> (none); Mnf. (none) -> EXV107M016A9GAA; Notes 100u 35V 85C -> (none); Package ThroughHole:C_Radial_D6.3_L11.2_P2.5 -> (none); Price 0.235€ -> 0.443
- JP1, JP2, JP3, JP4, JP5, JP6: footprint Pin_Headers:Pin_Header_Straight_1x02 -> Resistors_SMD:R_0805_HandSoldering; Distributor SparkFun PRT-12791 -> (none); Manufacturer - -> (none); Mnf. (none) -> CRCW08050000Z0EA; Notes https://www.sparkfun.com/products/12791 -> (none); Package 2x23 pin male PTH header -> (none); Price - -> 0.094
- P2, P4: Distributor SparkFun PRT-12791 -> (none); Manufacturer - -> (none); Notes https://www.sparkfun.com/products/12791 -> (none); Package 2x23 pin male PTH header -> (none); Price - -> (none)
- P7, P8: footprint Connect:bornier4 -> satnogs:MKDS_1.5-4; Distributor SparkFun PRT-08432 -> (none); Manufacturer - -> (none); Mnf. (none) -> Phoenix 1985467; Notes https://www.sparkfun.com/products/8432 -> (none); Package 5mm Pitch 4-Pin -> (none); Price 1.8€ -> 0.7
- R1: Distributor Mouser 71-CRCW0805120RJNEA -> (none); Manufacturer CRCW0805120RJNEA -> (none); Mnf. (none) -> CRCW0805120RJNEA; Notes 1/8W 5% -> (none); Package 0805 -> (none); Price 0.091€ -> 0.091
- R2, R3, R5, R6: Distributor Mouser 71-CRCW0805J-4.7K-E3 -> (none); Manufacturer CRCW08054K70JNEA -> (none); Mnf. (none) -> CRCW08054K70JNEA; Notes 1/8W 5% -> (none); Package 0805 -> (none); Price 0.091€ -> 0.091
- R4, R7: Distributor Mouser 71-CRCW0805J-100K-E3 -> (none); Manufacturer CRCW0805100KJNEA -> (none); Mnf. (none) -> CRCW0805100KJNEA; Notes 1/8W 5% -> (none); Package 0805 -> (none); Price 0.091€ -> 0.091
- R8, R9: value 4.7k -> 10; Distributor Mouser 71-CRCW0805J-4.7K-E3 -> (none); Manufacturer CRCW08054K70JNEA -> (none); Mnf. (none) -> CRCW080510R0JNEA; Notes 1/8W 5% -> (none); Package 0805 -> (none); Price 0.091€ -> 0.091
Connections:
- net labels added: +12V, BOOT, COMP, CTS, DTR, FB, M1D1, M1D2, M1RST, M1SF, M1SLP, M2D1, M2D2, M2RST, M2SF, M2SLP, MS2M1, MS2M2, MS3M1, MS3M2, PB4, PB5, RT/CLK, SCL, SCL0, SDA, SDA0, SW, SW_VIN
- net labels removed: SCL2, SDA2, SF, VMOT
- wire segments 153 -> 229
- no-connect marks 6 -> 10
Other:
- note added: "Always follow NEC guidelines for applying low-voltage fuses. Generally,\nthe MINIMUM fuse size should be based on 125% of the circuits full load\ncurrent. Time-delay fuses should be used for inductive loads."
- note added: "D2 is for inverse voltage protection"
- note added: "D4 is optional, for transient voltage suppressor"
- note added: "Debouncing filter\nfor the mechanichal\nend-stops.\nhttp://wot.lv/combating-endstop-noise-on-a-reprap.html\n"
- note added: "GND Pad for box shielding"
- note added: "M1IN1->STEPM1->D6\nM1IN2->DIRM1->D5\nM2IN1->STEPM2->D10\nM2IN2->DIRM2->D9\nSLEW/INV default state: GND"
- note added: "Note for microstepping\nMS1 MS2 MS3 Microstep\nLow Low Low Full\nHigh Low Low Half\nLow High Low Quarter\nHigh High Low Eighth\nHigh High High Sixteenth"
- note added: "Power Supply Module"
- note added: "RS-485 and power supply have Common GND.\nRS-485 requires ground wire to equalize node\nvoltage differences."
- note added: "Regulator in pro-mini, is MIC5205:\n5V@150mA with reverse-current protection\nFilter switching regulator\nfor 5V LDO. Cut 440kHz of switching regulator."
- note added: "Solder to have UART\nas communication"
- note added: "Stepper Motors"
- note added: "The characteristic impedance of UTP CAT5, CAT6\nis around 100ohm. With 120ohm termination in both\nsides, may get good results with these cables\n(Must be within 20%)."
- note added: "VIN: 20 - 60V"
- note added: "Vout: 12V@3A"
- note added: "\nFor distance problems, use P82B715\nI2C extender (for now we don't need)"
- note removed: "Dev pins"
- note removed: "EndStops"
- note removed: "Failsafe-biasing network for \nlegacy transceivers like SP485CN-L\n"
- note removed: "I2C-1,2"
- note removed: "M1IN1->DIRM1->D6\nM1IN2->STEPM1->D5\nM2IN1->DIRM2-D10\nM2IN2->STEPM2->D9"
- note removed: "Microcontroller"
- note removed: "Power In for stepper motors"
- note removed: "RS485"
- note removed: "Regulator in pro-mini, is MIC5205:\n5V@150mA with reverse-current protection"
- note removed: "Stepper motor 1"
- note removed: "Stepper motor 2"
- moved on the sheet: C1, C3, C4, JP1, JP2, JP3, JP4, JP5, JP6, P2, P4, P7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
